File: Electronics/PRoMo_v0_2/Communication.sch (KiCad schematic (older format))
At the start: 16 parts, among them J23 USB_B_Micro, J24 Conn_01x02, U10 NRF24L01_Breakout, U11 FT232RL

Commit message: Start working on HW v0.2
Parts:
- added TP6, TP7: TestPoint, TestPoint:TestPoint_Pad_D1.5mm, symbol Connector:TestPoint
- renumbered C36 to C28, C37 to C29, C38 to C30, C39 to C31, C40 to C32, D19 to D13, D20 to D14, D21 to D15, J23 to J13, J24 to J14, R25 to R15, R26 to R16, TP6 to TP8
Connections:
- net FTDI_RX: now also U11.1 (TXD), TP6.1; no longer U11.5 (RXD)
- net FTDI_TX: now also U11.5 (RXD), TP7.1; no longer U11.1 (TXD)
- net SPI2_MISO renamed NRF_SPI_MISO
- net SPI2_MOSI renamed NRF_SPI_MOSI
- net SPI2_SCK renamed NRF_SPI_SCK
Other:
- moved on the sheet: D14, D15, R15, R16
