File: Electronics/PRoMo_v0_2/Motor_driver.sch (KiCad schematic (older format))
At the start: 11 parts, among them J16 ME_L, J17 ME_R, U7 DRV8833PWP

Commit message: Small update to schematic and todo
Parts:
- added J25: Motor_power, Connector_PinHeader_2.54mm:PinHeader_1x02_P2.54mm_Vertical, symbol Connector_Generic:Conn_01x02
Connections:
- net NRST: now also J25.2 (Pin_2); no longer U7.1 (nSLEEP)
- new net: J25.1 (Pin_1), U7.1 (nSLEEP)
Other:
- moved on the sheet: R20
Changed lines of the file:
@@
 L Device:R_Small R?
 U 1 1 5F9E817E
-P 4450 2850
+P 4450 2300
 AR Path="/5F9E817E" Ref="R?"  Part="1"
 AR Path="/5F9DA82B/5F9E817E" Ref="R20"  Part="1"
-F 0 "R20" H 4509 2896 50  0000 L CNN
-F 1 "47k" H 4509 2805 50  0000 L CNN
-F 2 "Resistor_SMD:R_0805_2012Metric_Pad1.15x1.40mm_HandSolder" H 4450 2850 50  0001 C CNN
-F 3 "~" H 4450 2850 50  0001 C CNN
-F 4 "C17713" H 4450 2850 50  0001 C CNN "LCSC"
-F 5 "Basic" H 4450 2850 50  0001 C CNN "Catalog"
-	1    4450 2850
+F 0 "R20" H 4509 2346 50  0000 L CNN
+F 1 "47k" H 4509 2255 50  0000 L CNN
+F 2 "Resistor_SMD:R_0805_2012Metric_Pad1.15x1.40mm_HandSolder" H 4450 2300 50  0001 C CNN
+F 3 "~" H 4450 2300 50  0001 C CNN
+F 4 "C17713" H 4450 2300 50  0001 C CNN "LCSC"
+F 5 "Basic" H 4450 2300 50  0001 C CNN "Catalog"
+	1    4450 2300
 	1    0    0    -1
 $EndComp
@@
 L power:+3V3 #PWR?
 U 1 1 5F9E8184
-P 4450 2650
+P 4450 2100
 AR Path="/5F9E8184" Ref="#PWR?"  Part="1"
 AR Path="/5F9DA82B/5F9E8184" Ref="#PWR096"  Part="1"
-F 0 "#PWR096" H 4450 2500 50  0001 C CNN
-F 1 "+3V3" H 4465 2823 50  0000 C CNN
-F 2 "" H 4450 2650 50  0001 C CNN
-F 3 "" H 4450 2650 50  0001 C CNN
-	1    4450 2650
-	1    0    0    -1
-$EndComp
-Wire Wire Line
-	4450 2650 4450 2750
-Wire Wire Line
-	4450 2950 4450 3050
+F 0 "#PWR096" H 4450 1950 50  0001 C CNN
+F 1 "+3V3" H 4465 2273 50  0000 C CNN
+F 2 "" H 4450 2100 50  0001 C CNN
+F 3 "" H 4450 2100 50  0001 C CNN
+	1    4450 2100
+	1    0    0    -1
+$EndComp
+Wire Wire Line
+	4450 2100 4450 2200
+Wire Wire Line
+	4450 2400 4450 2500
 Wire Wire Line
 	4450 3150 4550 3150
@@
 Text GLabel 4250 3950 0    50   Input ~ 0
 MR_PWM_L
-Text Label 4700 2350 2    50   ~ 0
+Text Label 3250 2100 2    50   ~ 0
 VM
 Wire Wire Line
@@
 	5150 4300 5150 4250
 Connection ~ 5100 4300
-Text GLabel 4200 2350 0    50   Input ~ 0
+Text GLabel 2750 2100 0    50   Input ~ 0
 VBAT
 Wire Wire Line
-	4200 2350 4700 2350
+	2750 2100 3250 2100
 NoConn ~ 5950 3450
 $Comp
@@
 Wire Wire Line
 	3550 3450 3550 3600
-Text GLabel 4250 3050 0    50   Input ~ 0
+Text GLabel 4250 2500 0    50   Input ~ 0
 NRST
 Wire Wire Line
-	4250 3050 4450 3050
-Connection ~ 4450 3050
-Wire Wire Line
-	4450 3050 4450 3150
+	4250 2500 4450 2500
+$Comp
+L Connector_Generic:Conn_01x02 J25
+U 1 1 602EE7A8
+P 4250 2900
+F 0 "J25" H 4150 2700 50  0000 C CNN
+F 1 "Motor_power" H 4450 2700 50  0000 C CNN
+F 2 "Connector_PinHeader_2.54mm:PinHeader_1x02_P2.54mm_Vertical" H 4250 2900 50  0001 C CNN
+F 3 "~" H 4250 2900 50  0001 C CNN
+	1    4250 2900
+	-1   0    0    1
+$EndComp
+Wire Wire Line
+	4450 3150 4450 2900
+Wire Wire Line
+	4450 2800 4450 2500
+Connection ~ 4450 2500
 $EndSCHEMATC

Commit message: Start working on HW v0.2
Parts:
- removed J25: Motor_power, Connector_PinHeader_2.54mm:PinHeader_1x02_P2.54mm_Vertical, symbol Connector_Generic:Conn_01x02
- removed JP26, JP27: SolderJumper_2_Bridged, Jumper:SolderJumper-2_P1.3mm_Bridged_Pad1.0x1.5mm, symbol Jumper:SolderJumper_2_Bridged
- removed R20: 47k, Resistor_SMD:R_0805_2012Metric_Pad1.15x1.40mm_HandSolder, symbol Device:R_Small
- added JP2, JP3: SolderJumper_2_Open, Jumper:SolderJumper-2_P1.3mm_Open_Pad1.0x1.5mm, symbol Jumper:SolderJumper_2_Open
- added JP4: SolderJumper_3_Bridged12, Jumper:SolderJumper-3_P1.3mm_Bridged12_Pad1.0x1.5mm, symbol Jumper:SolderJumper_3_Bridged12
- renumbered C30 to C22, C31 to C23, C32 to C24, J16 to J6, J17 to J7, R19 to R10, R18 to R9
Connections:
- net GND: now also JP2.1 (A), JP3.1 (A)
- net NRST: now also JP4.3 (B)
- net at U7.1 (nSLEEP): now also JP4.2 (C)
- net ADC_ML_SENSE: now reaches R9.1, U7.3 (AISEN)
- net ADC_ML_SENSE: now also JP2.2 (B)
- net ADC_MR_SENSE: now reaches R10.1, U7.6 (BISEN)
- net ADC_MR_SENSE: now also JP3.2 (B)
- new net DRV_EN: JP4.1 (A)
Other:
- moved on the sheet: R10, R9
