File: Electronics/PRoMo_v0_2/PRoMo.kicad_pcb (KiCad board)
At the start: 2 copper layers, 100 x 100 mm, 154 parts, among them J1 AN14, J10 SPI1_AUX, J11 I2C2_AUX, J12 Conn_01x02, J13 Conn_01x02, J14 Conn_01x02, J15 Conn_01x02, J16 ME_L, J17 ME_R, J18 Conn_01x02, J19 Conn_02x02_Counter_Clockwise, J2 GPIO1, J20 Conn_02x02_Counter_Clockwise, J21 AUX_IN, J22 AUX_OUT, J23 USB_B_Micro, J24 Conn_01x02, J3 GPIO2, J4 GPIO3, J5 AN8, J6 AN9, J7 AN15, J8 Programming, J9 UART6_AUX, SW1 RESET_BP, SW2 WKP_BP, SW3 SW_SPDT, U1 STM32F405RGTx, U10 NRF24L01_Breakout, U11 FT232RL, U2 VL53l0x_breakout, U3 VL53l0x_breakout, U4 VL53l0x_breakout, U5 VL53l0x_breakout, U6 MPU-6050, U7 DRV8833PWP, U8 LM2596S-5, U9 AMS1117-3.3, Y1 Crystal_GND24

Commit message: Start working on HW v0.2
Parts:
- removed C33: 680uF, Capacitor_THT:CP_Radial_D6.3mm_P2.50mm
- removed C34: 220uF, Capacitor_THT:CP_Radial_D6.3mm_P2.50mm
- removed C35: 10uF, Capacitor_Tantalum_SMD:CP_EIA-3216-18_Kemet-A_Pad1.58x1.35mm_HandSolder
- removed C36: 100uF, Capacitor_THT:CP_Radial_D6.3mm_P2.50mm
- removed C37, C39: 100nF, Capacitor_SMD:C_0805_2012Metric_Pad1.15x1.40mm_HandSolder
- removed C38: Unpopulated, Capacitor_SMD:C_0805_2012Metric_Pad1.15x1.40mm_HandSolder
- removed C40: 4.7uF, Capacitor_SMD:C_0805_2012Metric_Pad1.15x1.40mm_HandSolder
- removed D16: LED_Yellow, LED_SMD:LED_0805_2012Metric_Pad1.15x1.40mm_HandSolder
- removed D17, D18: LED_Green, LED_SMD:LED_0805_2012Metric_Pad1.15x1.40mm_HandSolder
- removed D19: D_Zener_Small, Diode_SMD:D_SMA_Handsoldering
- removed D20, D21: Yellow, LED_SMD:LED_0805_2012Metric_Pad1.15x1.40mm_HandSolder
- removed J15, J18, J24: Conn_01x02, Connector_PinHeader_2.54mm:PinHeader_1x02_P2.54mm_Vertical
- removed J16: ME_L, Connector_PinHeader_2.54mm:PinHeader_1x06_P2.54mm_Vertical
- removed J17: ME_R, Connector_PinHeader_2.54mm:PinHeader_1x06_P2.54mm_Vertical
- removed J19, J20: Conn_02x02_Counter_Clockwise, Connector_PinSocket_2.54mm:PinSocket_2x02_P2.54mm_Vertical
- removed J21: AUX_IN, Connector_PinHeader_2.54mm:PinHeader_1x02_P2.54mm_Vertical
- removed J22: AUX_OUT, Connector_PinHeader_2.54mm:PinHeader_1x02_P2.54mm_Vertical
- removed J23: USB_B_Micro, Connector_USB:USB_Micro-B_Molex_47346-0001
- removed JP10, JP23, JP24, JP5, JP6: SolderJumper_3_Bridged12, Jumper:SolderJumper-3_P1.3mm_Bridged12_Pad1.0x1.5mm
- removed JP11, JP14, JP15, JP16, JP17, JP18, JP19, JP20, JP21, JP22, JP26, JP27, JP7, JP8, JP9: SolderJumper_2_Bridged, Jumper:SolderJumper-2_P1.3mm_Bridged_Pad1.0x1.5mm
- removed JP12, JP13: SolderJumper_2_Open, Jumper:SolderJumper-2_P1.3mm_Open_Pad1.0x1.5mm
- removed JP25: SLAVE_ADDR, Jumper:SolderJumper-3_P1.3mm_Bridged12_Pad1.0x1.5mm
- removed R17: 1k, Resistor_SMD:R_0805_2012Metric_Pad1.15x1.40mm_HandSolder
- removed R18, R19: Sense, Resistor_SMD:R_2512_6332Metric_Pad1.52x3.35mm_HandSolder
- removed R20: 47k, Resistor_SMD:R_0805_2012Metric_Pad1.15x1.40mm_HandSolder
- removed R21: 470R, Resistor_SMD:R_0805_2012Metric_Pad1.15x1.40mm_HandSolder
- removed R22: 330R, Resistor_SMD:R_0805_2012Metric_Pad1.15x1.40mm_HandSolder
- removed R23, R25, R26: 220R, Resistor_SMD:R_0805_2012Metric_Pad1.15x1.40mm_HandSolder
- removed R24: 47R, Resistor_SMD:R_0805_2012Metric_Pad1.15x1.40mm_HandSolder
- added C17: 100nF, Capacitor_SMD:C_0805_2012Metric_Pad1.15x1.40mm_HandSolder, F.Cu at (340.1, -42.5)
- added C19: 100nF, Capacitor_SMD:C_0805_2012Metric_Pad1.15x1.40mm_HandSolder, F.Cu at (295.4, -77.8)
- added C21: 2.2nF, Capacitor_SMD:C_0805_2012Metric_Pad1.15x1.40mm_HandSolder, F.Cu at (302.2, -71.9)
- added C23: 2.2uF, Capacitor_SMD:C_0805_2012Metric_Pad1.15x1.40mm_HandSolder, F.Cu at (328.0, -5.60)
- added C24: 10uF, Capacitor_SMD:C_0805_2012Metric_Pad1.15x1.40mm_HandSolder, F.Cu at (332.8, -7.50)
- added C25: 680uF, Capacitor_THT:CP_Radial_D6.3mm_P2.50mm, F.Cu at (295.7, 30.4)
- added D11: LED_Green, LED_SMD:LED_0805_2012Metric_Pad1.15x1.40mm_HandSolder, F.Cu at (224.6, 53.0)
- added D12: LED_Green, LED_SMD:LED_0805_2012Metric_Pad1.15x1.40mm_HandSolder, F.Cu at (224.3, 58.5)
- added D13: D_Zener_Small, Diode_SMD:D_SMA_Handsoldering, F.Cu at (102.8, 38.6)
- added D5: SK6812, LED_SMD:LED_SK6812_PLCC4_5.0x5.0mm_P3.2mm, F.Cu at (322.8, -50.7)
- added D7: SK6812, LED_SMD:LED_SK6812_PLCC4_5.0x5.0mm_P3.2mm, F.Cu at (340.4, -51.0)
- added D9: LED_Red, LED_SMD:LED_0805_2012Metric_Pad1.15x1.40mm_HandSolder, F.Cu at (224.9, 42.0)
- added SW4: SW_SPDT, Button_Switch_SMD:SW_SPDT_PCM12, F.Cu at (275.6, 66.4)
- added TP8: TestPoint, TestPoint:TestPoint_Pad_D1.5mm, F.Cu at (127.3, 25.9)
- C1: value 100nF -> 18pF
- C10: value 100nF -> 10uF
- C11: value 10uF -> 1uF
- C12: value 1uF -> 100nF
- C13, C28: value 100nF -> 100uF; footprint Capacitor_SMD:C_0805_2012Metric_Pad1.15x1.40mm_HandSolder -> Capacitor_THT:CP_Radial_D6.3mm_P2.50mm
- C14: value 4.7uF -> 100nF
- C15: value 100uF -> 100nF; footprint Capacitor_THT:CP_Radial_D6.3mm_P2.50mm -> Capacitor_SMD:C_0805_2012Metric_Pad1.15x1.40mm_HandSolder
- C18, C22: value 100nF -> 10nF
- C26: value 10nF -> 220uF; footprint Capacitor_SMD:C_0805_2012Metric_Pad1.15x1.40mm_HandSolder -> Capacitor_THT:CP_Radial_D6.3mm_P2.50mm
- C27: value 100nF -> 10uF; footprint Capacitor_SMD:C_0805_2012Metric_Pad1.15x1.40mm_HandSolder -> Capacitor_Tantalum_SMD:CP_EIA-3216-18_Kemet-A_Pad1.58x1.35mm_HandSolder
- C29: value 2.2nF -> 100nF
- C3: value 18pF -> 100nF
- C30: value 10nF -> Unpopulated
- C31, C8: value 2.2uF -> 100nF
- C32: value 10uF -> 4.7uF
- C6: value 2.2uF -> 4.7uF
- D10: value SK6812 -> LED_Yellow; footprint LED_SMD:LED_SK6812_PLCC4_5.0x5.0mm_P3.2mm -> LED_SMD:LED_0805_2012Metric_Pad1.15x1.40mm_HandSolder
- D14: value SS14 -> Yellow; footprint Diode_SMD:D_SMA_Handsoldering -> LED_SMD:LED_0805_2012Metric_Pad1.15x1.40mm_HandSolder
- D15: value LED_Red -> Yellow
- D8: value SK6812 -> SS14; footprint LED_SMD:LED_SK6812_PLCC4_5.0x5.0mm_P3.2mm -> Diode_SMD:D_SMA_Handsoldering
- H1, H2, H3, H4: footprint MountingHole:MountingHole_2.7mm_M2.5 -> MountingHole:MountingHole_3.2mm_M3
- J1: value AN14 -> Conn_01x02; footprint Connector_PinHeader_2.54mm:PinHeader_1x03_P2.54mm_Vertical -> Connector_PinHeader_2.54mm:PinHeader_1x02_P2.54mm_Vertical
- J10: value SPI1_AUX -> Conn_02x02_Counter_Clockwise; footprint Connector_PinHeader_2.54mm:PinHeader_1x06_P2.54mm_Vertical -> Connector_PinSocket_2.54mm:PinSocket_2x02_P2.54mm_Vertical
- J11: value I2C2_AUX -> AUX_IN; footprint Connector_PinHeader_2.54mm:PinHeader_1x04_P2.54mm_Vertical -> Connector_PinHeader_2.54mm:PinHeader_1x02_P2.54mm_Vertical
- J12: value Conn_01x02 -> AUX_OUT
- J13: value Conn_01x02 -> USB_B_Micro; footprint Connector_PinHeader_2.54mm:PinHeader_1x02_P2.54mm_Vertical -> Connector_USB:USB_Micro-B_Molex_47346-0001
- J2: value GPIO1 -> Conn_01x02; footprint Connector_PinHeader_2.54mm:PinHeader_1x03_P2.54mm_Vertical -> Connector_PinHeader_2.54mm:PinHeader_1x02_P2.54mm_Vertical
- J3: value GPIO2 -> Conn_01x02; footprint Connector_PinHeader_2.54mm:PinHeader_1x03_P2.54mm_Vertical -> Connector_PinHeader_2.54mm:PinHeader_1x02_P2.54mm_Vertical
- J4: value GPIO3 -> Conn_01x02; footprint Connector_PinHeader_2.54mm:PinHeader_1x03_P2.54mm_Vertical -> Connector_PinHeader_2.54mm:PinHeader_1x02_P2.54mm_Vertical
- J5: value AN8 -> Conn_01x03
- J6: value AN9 -> ME_L; footprint Connector_PinHeader_2.54mm:PinHeader_1x03_P2.54mm_Vertical -> Connector_PinHeader_2.54mm:PinHeader_1x06_P2.54mm_Vertical
- J7: value AN15 -> ME_R; footprint Connector_PinHeader_2.54mm:PinHeader_1x03_P2.54mm_Vertical -> Connector_PinHeader_2.54mm:PinHeader_1x06_P2.54mm_Vertical
- J8: value Programming -> Conn_01x02; footprint Connector_PinHeader_2.54mm:PinHeader_1x06_P2.54mm_Vertical -> Connector_PinHeader_2.54mm:PinHeader_1x02_P2.54mm_Vertical
- J9: value UART6_AUX -> Conn_02x02_Counter_Clockwise; footprint Connector_PinHeader_2.54mm:PinHeader_1x06_P2.54mm_Vertical -> Connector_PinSocket_2.54mm:PinSocket_2x02_P2.54mm_Vertical
- JP1: value SolderJumper_3_Bridged12 -> SLAVE_ADDR
- JP2, JP3: value SolderJumper_3_Bridged12 -> SolderJumper_2_Open; footprint Jumper:SolderJumper-3_P1.3mm_Bridged12_Pad1.0x1.5mm -> Jumper:SolderJumper-2_P1.3mm_Open_Pad1.0x1.5mm
- R10, R9: value 1k -> Sense; footprint Resistor_SMD:R_0805_2012Metric_Pad1.15x1.40mm_HandSolder -> Resistor_SMD:R_2512_6332Metric_Pad1.52x3.35mm_HandSolder
- R11: value 10k -> 470R
- R12: value 47R -> 330R
- R13: value 47R -> 220R
- R14: value 10k -> 47R
- R15, R16: value 1k -> 220R
- R2, R3: value 1k -> 10k
- R4, R5: value 1k -> 47R
- R8: value Unpopulated -> 1k
- SW1: value RESET_BP -> DIP-BUTTON_2P-6.0X3.0X4.3MM_; footprint Button_Switch_THT:SW_TH_Tactile_Omron_B3F-10xx -> Button_Switch_THT:SW_PUSH_6mm_H5mm
- SW2: value WKP_BP -> DIP-BUTTON_2P-6.0X3.0X4.3MM_; footprint Button_Switch_THT:SW_TH_Tactile_Omron_B3F-10xx -> Button_Switch_THT:SW_PUSH_6mm_H5mm
- SW3: value SW_SPDT -> DIP-BUTTON_2P-6.0X3.0X4.3MM_; footprint Button_Switch_SMD:SW_SPDT_PCM12 -> Button_Switch_THT:SW_PUSH_6mm_H5mm
- U1: value STM32F405RGTx -> STM32F401RETx
- moved J5 301.0 mm to (348.1, -53.0)
- moved C20 290.7 mm to (302.1, -77.1), turned to 0 degrees
- moved TP3 280.3 mm to (344.4, -59.5), turned to 0 degrees
- moved H4 252.8 mm to (258.6, -90.1)
- moved C22 249.7 mm to (328.1, -10.6), turned to 0 degrees
- moved J6 239.9 mm to (299.1, -11.2)
- moved U6 239.2 mm to (295.8, -71.7)
- moved H3 238.9 mm to (247.8, -90.1)
- moved C18 237.1 mm to (290.0, -78.5)
- moved R9 233.0 mm to (328.9, 2.80)
- moved D6 232.9 mm to (331.6, -51.0)
- moved D8 231.3 mm to (313.4, 55.1), turned to 0 degrees
- moved U7 224.0 mm to (320.1, -7.92), turned to 0 degrees
- moved C14 223.0 mm to (313.9, -42.9), turned to 0 degrees
- moved H1 219.4 mm to (229.3, -89.7)
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Connections:
- net SPI2_MISO renamed NRF_SPI_MISO
- net SPI2_MOSI renamed NRF_SPI_MOSI
- net SPI2_SCK renamed NRF_SPI_SCK
- C1 pad 1: /NRST -> Net-(C1-Pad1)
- C10 pad 1: Net-(C10-Pad1) -> +3V3
- C10 pad 2: +3V3 -> GND
- C13 pad 1: +3V3 -> +5V
- C16 pad 1: Net-(C16-Pad1) -> +5V
- C18 pad 1: +5V -> GND
- C18 pad 2: GND -> +3V3
- C20 pad 1: +5V -> Net-(C20-Pad1)
- C22 pad 1: +5V -> Net-(C22-Pad1)
- C22 pad 2: GND -> VBAT
- C26 pad 1: GND -> +5V
- C26 pad 2: +3V3 -> GND
- C27 pad 1: GND -> +3V3
- C27 pad 2: +3V3 -> GND
- C28 pad 1: Net-(C28-Pad1) -> +3V3
- C29 pad 1: Net-(C29-Pad1) -> GND
- C29 pad 2: GND -> Net-(C29-Pad2)
- C3 pad 1: Net-(C3-Pad1) -> +3V3
- C30 pad 1: Net-(C30-Pad1) -> +3V3
- C30 pad 2: VBAT -> GND
- C31 pad 2: Net-(C31-Pad2) -> +5V
- C32 pad 1: VBAT -> GND
- C32 pad 2: GND -> +5V
- C4 pad 1: +3V3 -> NRST
- C8 pad 1: Net-(C8-Pad1) -> +3V3
- C9 pad 1: +3V3 -> Net-(C9-Pad1)
- C9 pad 2: GND -> +3V3
- D14 pad 2: GND -> Net-(D14-Pad2)
- D15 pad 1: GND -> Net-(D15-Pad1)
- D3 pad 1: Net-(C16-Pad1) -> Net-(C14-Pad1)
- D4 pad 3: Net-(C16-Pad1) -> Net-(C14-Pad1)
- D6 pad 2: Net-(D4-Pad4) -> Net-(D5-Pad4)
- D8 pad 1: GND -> Net-(D8-Pad1)
- D8 pad 2: Net-(D6-Pad4) -> GND
- J1 pad 1: Net-(J1-Pad1) -> VL53l0_1_XSHUT
- J1 pad 2: Net-(J1-Pad2) -> GND
- J10 pad 1: Net-(J10-Pad1) -> +3V3
- J10 pad 2: SPI1_NSS -> +3V3
- J10 pad 3: SPI1_SCK -> GND
- J10 pad 4: SPI1_MISO -> GND
- J11 pad 1: Net-(J11-Pad1) -> GND
- J11 pad 2: I2C2_SDA -> VBAT
- J12 pad 1: VL53l0_1_XSHUT -> GND
- J12 pad 2: GND -> +5V
- J13 pad 1: VL53l0_2_XSHUT -> VBUS
- J13 pad 2: GND -> Net-(J13-Pad2)
- J14 pad 1: VL53l0_3_XSHUT -> +5V
- J14 pad 2: GND -> Net-(D13-Pad1)
- J2 pad 1: Net-(J2-Pad1) -> VL53l0_2_XSHUT
- J2 pad 2: Servo1 -> GND
- J3 pad 1: Net-(J3-Pad1) -> VL53l0_3_XSHUT
- J3 pad 2: Servo2 -> GND
- J4 pad 1: Net-(J4-Pad1) -> VL53l0_4_XSHUT
- J4 pad 2: Servo3 -> GND
- J5 pad 1: Net-(J5-Pad1) -> +5V
- J5 pad 2: Net-(J5-Pad2) -> Net-(D7-Pad4)
- J6 pad 1: Net-(J6-Pad1) -> /Motor_driver/ML1
- J6 pad 2: Net-(J6-Pad2) -> /Motor_driver/ML2
- J6 pad 3: GND -> +3V3
- J7 pad 1: Net-(J7-Pad1) -> /Motor_driver/MR1
- J7 pad 2: Net-(J7-Pad2) -> /Motor_driver/MR2
- J7 pad 3: GND -> +3V3
- J8 pad 1: +3V3 -> GND
- J8 pad 2: /TCK -> Net-(J8-Pad2)
- J9 pad 1: Net-(J9-Pad1) -> +5V
- J9 pad 2: UART6_RX -> +5V
- J9 pad 3: UART6_TX -> GND
- J9 pad 4: +3V3 -> GND
- JP1 pad 1: +3V3 -> GND
- JP1 pad 2: Net-(J1-Pad1) -> Net-(JP1-Pad2)
- JP1 pad 3: +5V -> +3V3
- JP2 pad 1: +3V3 -> GND
- JP2 pad 2: Net-(J2-Pad1) -> ADC_ML_SENSE
- JP3 pad 1: +3V3 -> GND
- JP3 pad 2: Net-(J3-Pad1) -> ADC_MR_SENSE
- JP4 pad 1: +3V3 -> DRV_EN
- JP4 pad 2: Net-(J4-Pad1) -> Net-(JP4-Pad2)
- JP4 pad 3: +5V -> NRST
- L1 pad 1: Net-(D14-Pad1) -> Net-(D8-Pad1)
- L2 pad 1: Net-(D14-Pad1) -> Net-(D8-Pad1)
- R1 pad 1: ADC1_14 -> +3V3
- R1 pad 2: Net-(J1-Pad2) -> I2C_AUX_SDA
- R10 pad 1: GND -> ADC_MR_SENSE
- R10 pad 2: ADC1_15 -> GND
- R11 pad 1: Net-(R11-Pad1) -> Net-(D9-Pad2)
- R11 pad 2: GND -> VBAT
- R12 pad 1: +3V3 -> Net-(D10-Pad2)
- R12 pad 2: Net-(D1-Pad2) -> VBUS
- R13 pad 1: +3V3 -> Net-(D11-Pad2)
- R13 pad 2: Net-(D2-Pad2) -> +5V
- R14 pad 1: GND -> Net-(D12-Pad2)
- R14 pad 2: Net-(JP19-Pad2) -> +3V3
- R15 pad 1: +3V3 -> +5V
- R15 pad 2: I2C2_SCL -> Net-(D14-Pad2)
- R16 pad 1: +3V3 -> +5V
- R16 pad 2: I2C1_SCL -> Net-(D15-Pad2)
- R2 pad 1: ADC1_8 -> /BOOT1_BP2
- R2 pad 2: Net-(J5-Pad2) -> +3V3
- R3 pad 1: ADC1_9 -> /BP1
- R3 pad 2: Net-(J6-Pad2) -> +3V3
- R4 pad 1: GND -> +3V3
- R4 pad 2: ADC1_14 -> Net-(D1-Pad2)
- R5 pad 1: GND -> +3V3
- R5 pad 2: ADC1_8 -> Net-(D2-Pad2)
- R6 pad 1: GND -> +3V3
- R6 pad 2: ADC1_9 -> I2C_AUX_SCL
- R7 pad 1: ADC1_15 -> +3V3
- R7 pad 2: Net-(J7-Pad2) -> VL53l0_I2C_SCL
- R8 pad 2: /NRST -> VL53l0_I2C_SDA
- R9 pad 1: +3V3 -> ADC_ML_SENSE
- R9 pad 2: I2C2_SDA -> GND
- SW1 pad 1: /NRST -> GND
- SW1 pad 2: GND -> NRST
- SW2 pad 1: Net-(JP19-Pad2) -> /BP1
- SW2 pad 2: +3V3 -> GND
- SW3 pad 1: Net-(SW3-Pad1) -> /BOOT1_BP2
- SW3 pad 2: Net-(J18-Pad2) -> GND
- TP1 pad 1: Net-(C14-Pad1) -> Net-(TP1-Pad1)
- TP3 pad 1: Net-(TP3-Pad1) -> Net-(D7-Pad4)
- TP6 pad 1: Net-(TP6-Pad1) -> FTDI_RX
- TP7 pad 1: Net-(D10-Pad4) -> FTDI_TX
- U1 pad 1: Net-(C10-Pad1) -> Net-(C9-Pad1)
- U1 pad 10: Net-(JP16-Pad1) -> ADC_ML_SENSE
- U1 pad 11: Net-(JP17-Pad1) -> ADC_MR_SENSE
- U1 pad 14: Net-(JP19-Pad1) -> PWM_ML_H
- U1 pad 15: Net-(JP20-Pad1) -> PWM_ML_L
- U1 pad 16: MR_PWM_H -> PWM_MR_H
- U1 pad 17: MR_PWM_L -> PWM_MR_L
- U1 pad 2: MPU_FSYNC -> /BP1
- U1 pad 20: SPI1_NSS -> SPI_AUX_NSS
- U1 pad 21: SPI1_SCK -> SPI_AUX_SCK
- U1 pad 22: SPI1_MISO -> SPI_AUX_MISO
- U1 pad 23: SPI1_MOSI -> SPI_AUX_MOSI
- U1 pad 24: ADC1_14 -> AUX_SPI_INT
- U1 pad 25: ADC1_15 -> /BATT_ADC
- U1 pad 26: ADC1_8 -> /AUX_GPIO_1
- U1 pad 27: ADC1_9 -> /AUX_GPIO_2
- U1 pad 28: NRF_IRQ -> /BOOT1_BP2
- U1 pad 3: MPU_INT -> VL53l0_3_XSHUT
- U1 pad 30: Net-(C14-Pad1) -> Net-(C6-Pad1)
- U1 pad 31: Net-(C6-Pad1) -> GND
- U1 pad 37: UART6_TX -> AUX_UART_TX
- U1 pad 38: UART6_RX -> AUX_UART_RX
- U1 pad 39: Net-(JP18-Pad1) -> I2C_AUX_INT
- U1 pad 4: VL53l0_1_INT -> VL53l0_4_XSHUT
- U1 pad 40: I2C2_SDA -> I2C_AUX_SDA
- U1 pad 41: I2C2_SCL -> I2C_AUX_SCL
- U1 pad 42: FTDI_TX -> USB_VBUS
- U1 pad 43: FTDI_RX -> /LED_USR2
- U1 pad 44: FTDI_CTS -> USB_DM
- U1 pad 45: FTDI_RTS -> USB_DP
- U1 pad 46: /TMS -> /SWIO
- U1 pad 47: Net-(C8-Pad1) -> GND
- U1 pad 49: /TCK -> /SWCLK
- U1 pad 5: Net-(C2-Pad1) -> Net-(C1-Pad1)
- U1 pad 50: Net-(JP21-Pad1) -> VL53l0_1_INT
- U1 pad 51: Servo1 -> VL53l0_1_XSHUT
- U1 pad 52: Servo2 -> VL53l0_2_XSHUT
- U1 pad 53: Servo3 -> ADDR_LEDS
- U1 pad 54: ADDR_LEDS -> DRV_EN
- U1 pad 55: Net-(JP22-Pad1) -> /LED_USR1
- U1 pad 6: Net-(C3-Pad1) -> Net-(C2-Pad1)
- U1 pad 60: Net-(R11-Pad1) -> /BOOT0
- U1 pad 61: I2C1_SCL -> VL53l0_I2C_SCL
- U1 pad 62: I2C1_SDA -> VL53l0_I2C_SDA
- U1 pad 7: /NRST -> NRST
- U1 pad 8: Net-(JP14-Pad1) -> MPU_INT
- U1 pad 9: Net-(JP15-Pad1) -> NRF_IRQ
- U11 pad 1: FTDI_TX -> FTDI_RX
- U11 pad 10: Net-(U11-Pad10) -> (no net)
- U11 pad 11: FTDI_CTS -> (no net)
- U11 pad 12: Net-(U11-Pad12) -> (no net)
- U11 pad 13: Net-(U11-Pad13) -> (no net)
- U11 pad 14: Net-(U11-Pad14) -> (no net)
- U11 pad 15: Net-(J23-Pad3) -> Net-(J13-Pad3)
- U11 pad 16: Net-(J23-Pad2) -> Net-(J13-Pad2)
- U11 pad 17: Net-(C37-Pad2) -> Net-(C29-Pad2)
- U11 pad 2: Net-(TP6-Pad1) -> Net-(TP8-Pad1)
- U11 pad 22: Net-(D21-Pad1) -> Net-(D15-Pad1)
- U11 pad 23: Net-(D20-Pad1) -> Net-(D14-Pad1)
- U11 pad 26: Net-(U11-Pad26) -> (no net)
- U11 pad 27: Net-(U11-Pad27) -> (no net)
- U11 pad 28: Net-(U11-Pad28) -> (no net)
- U11 pad 3: FTDI_RTS -> (no net)
- U11 pad 5: FTDI_RX -> FTDI_TX
- U11 pad 6: Net-(U11-Pad6) -> (no net)
- U11 pad 9: Net-(U11-Pad9) -> (no net)
- U2 pad 3: I2C1_SCL -> VL53l0_I2C_SCL
- U2 pad 4: I2C1_SDA -> VL53l0_I2C_SDA
- U3 pad 3: I2C1_SCL -> VL53l0_I2C_SCL
- U3 pad 4: I2C1_SDA -> VL53l0_I2C_SDA
- U3 pad 5: Net-(TP2-Pad1) -> Net-(TP1-Pad1)
- U4 pad 3: I2C1_SCL -> VL53l0_I2C_SCL
- U4 pad 4: I2C1_SDA -> VL53l0_I2C_SDA
- U4 pad 5: Net-(TP3-Pad1) -> Net-(TP2-Pad1)
- U5 pad 3: I2C1_SCL -> VL53l0_I2C_SCL
- U5 pad 4: I2C1_SDA -> VL53l0_I2C_SDA
- U6 pad 1: Net-(U6-Pad1) -> (no net)
- U6 pad 10: Net-(C28-Pad1) -> Net-(C20-Pad1)
- U6 pad 20: Net-(C29-Pad1) -> Net-(C21-Pad1)
- U6 pad 23: I2C2_SCL -> AUX_I2C_SCL
- U6 pad 24: I2C2_SDA -> AUX_I2C_SDA
- U6 pad 6: Net-(U6-Pad6) -> (no net)
- U6 pad 7: Net-(U6-Pad7) -> (no net)
- U6 pad 9: Net-(JP25-Pad2) -> Net-(JP1-Pad2)
- U7 pad 1: Net-(R20-Pad2) -> Net-(JP4-Pad2)
- U7 pad 11: Net-(C30-Pad1) -> Net-(C22-Pad1)
- U7 pad 14: Net-(C31-Pad2) -> Net-(C23-Pad2)
- U7 pad 3: Net-(JP26-Pad2) -> ADC_ML_SENSE
- U7 pad 6: Net-(JP27-Pad2) -> ADC_MR_SENSE
- U8 pad 2: Net-(D14-Pad1) -> Net-(D8-Pad1)
- Y1 pad 1: Net-(C2-Pad1) -> Net-(C1-Pad1)
- Y1 pad 3: Net-(C3-Pad1) -> Net-(C2-Pad1)
Routing:
- net +3V3: track 608.5 -> 0.00 mm, vias 25 -> 0
- net +5V: track 358.4 -> 0.00 mm, vias 19 -> 0
- net I2C1_SCL: track 232.7 -> 0.00 mm, vias 6 -> 0
- net I2C1_SDA: track 228.0 -> 0.00 mm, vias 7 -> 0
- net Net-(D6-Pad4): track 118.4 -> 0.00 mm, vias 2 -> 0
- net GND: track 114.5 -> 0.00 mm, vias 140 -> 0
- net Net-(JP17-Pad1): track 109.7 -> 0.00 mm, vias 3 -> 0
- net VBAT: track 93.4 -> 0.00 mm, vias 2 -> 0
- net Net-(JP16-Pad1): track 84.8 -> 0.00 mm, vias 3 -> 0
- net ADC1_9: track 75.9 -> 0.00 mm, vias 4 -> 0
- net /NRST: track 66.9 -> 0.00 mm, vias 3 -> 0
- net FTDI_CTS: track 63.5 -> 0.00 mm, vias 2 -> 0
- net ADC1_8: track 63.3 -> 0.00 mm, vias 2 -> 0
- net FTDI_RX: track 60.2 -> 0.00 mm, vias 2 -> 0
- net FTDI_RTS: track 58.9 -> 0.00 mm, vias 2 -> 0
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- removed copper zone on B.Cu, net GND
- removed copper zone on F.Cu, net GND
Other:
- board outline removed
- board text removed: "3V3"
- board text removed: "5V"
- board text removed: "AIO14"
- board text removed: "AIO15"
- board text removed: "AIO8"
- board text removed: "AIO9"
- board text removed: "BATT"
- board text removed: "BP1"
- board text removed: "DIO10"
- board text removed: "DIO11"
- board text removed: "DIO12"
- board text removed: "GND"
- board text removed: "I2C"
- board text removed: "M1"
- board text removed: "M2"
- board text removed: "MD"
- board text removed: "MG"
- board text removed: "MI"
- board text removed: "MO"
- board text removed: "NSS"
- board text removed: "ON/OFF"
- board text removed: "PA"
- board text removed: "PB"
- board text removed: "PB0"
- board text removed: "PB1"
- board text removed: "PC10"
- board text removed: "PC11"
- board text removed: "PC12"
- board text removed: "PC4"
- board text removed: "PC5"
- board text removed: "PROG"
- board text removed: "PRoMo v1.0"
- board text removed: "RST"
- board text removed: "RX"
- board text removed: "SCK"
- board text removed: "SCL"
- board text removed: "SDA"
- board text removed: "SPI"
- board text removed: "TCK"
- board text removed: "TMS"
- board text removed: "TX"
- board text removed: "UART"
- board text removed: "VCC"
- board text removed: "VUSB"
