File: Electronics/PRoMo_v0_2/PRoMo.sch (KiCad schematic (older format))
At the start: 77 parts, among them J1 AN14, J10 SPI1_AUX, J11 I2C2_AUX, J2 GPIO1, J3 GPIO2, J4 GPIO3, J5 AN8, J6 AN9, J7 AN15, J8 Programming, J9 UART6_AUX, SW1 RESET_BP, SW2 WKP_BP, U1 STM32F405RGTx, Y1 Crystal_GND24

Commit message: Small update to schematic and todo
Other:
- note added: "DONE:\n - Add a jumper for motor power\n - Separate Shield and Ground from USB connector"
- note added: "TODO:\n - Change Button footprint\n - Add diode between power levels\n - Investigate why VBAT in back driven from 5V/3V3?\n - Less bright LEDs\n - Move TIM2 away from PA15 (default state high)\n - Move Mot/Coder header to the side of th motors (with mirrored orientation)\n - Add 2 ALED in front and move button\n - Add 1/2 ALED in the back\n - Wider holes for battery\n - Better positions for stand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"
- note removed: "DONE:\n - Separate Shield and Ground from USB connector"
- note removed: "TODO:\n - Change Button footprint\n - Add diode between power levels\n - Less bright LEDs\n - Move TIM2 away from PA15 (default state high)\n - Move Mot/Coder header to the side of th motors (with mirrored orientation)\n - Add 2 ALED in front and move button\n - Add 1/2 ALED in the back\n - Wider holes for battery\n - Better positions for standoffs\n - Maybe change aux header layout\n\n - Battery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"
Changed lines of the file:
@@
 NRST
 Text Notes 14550 3100 0    100  ~ 0
-TODO:\n - Change Button footprint\n - Add diode between power levels\n - Less bright LEDs\n - Move TIM2 away from PA15 (default state high)\n - Move Mot/Coder header to the side of th motors (with mirrored orientation)\n - Add 2 ALED in front and move button\n - Add 1/2 ALED in the back\n - Wider holes for battery\n - Better positions for standoffs\n - Maybe change aux header layout\n\n - Battery monitoring (bridge divider to ADC pin)\n - Power multiplexer (ex: TPS2113A) ???\n - Add test points or solder joint where not sure\n\n
+TODO:\n - Change Button footprint\n - Add diode between power levels\n - Investigate why VBAT in back driven from 5V/3V3?\n - Less bright LEDs\n - Move TIM2 away from PA15 (default state high)\n - Move Mot/Coder header to the side of th motors (with mirrored orientation)\n - Add 2 ALED in front and move button\n - Add 1/2 ALED in the back\n - Wider holes for battery\n - Better positions for standoffs\n - Maybe change aux header layout\n\n - Battery monitoring (bridge divider to ADC pin)\n - Power multiplexer (ex: TPS2113A) ???\n - Add test points or solder joint where not sure\n\n
 Text Notes 14550 3950 0    100  ~ 0
-DONE:\n - Separate Shield and Ground from USB connector
+DONE:\n - Add a jumper for motor power\n - Separate Shield and Ground from USB connector
 $EndSCHEMATC

Commit message: Start working on HW v0.2
Parts:
- removed C10: 100nF, Capacitor_SMD:C_0805_2012Metric_Pad1.15x1.40mm_HandSolder, symbol Device:C_Small
- removed C14: 4.7uF, Capacitor_SMD:C_0805_2012Metric_Pad1.15x1.40mm_HandSolder, symbol Device:C_Small
- removed C3: 18pF, Capacitor_SMD:C_0805_2012Metric_Pad1.15x1.40mm_HandSolder, symbol Device:C_Small
- removed C8: 2.2uF, Capacitor_SMD:C_0805_2012Metric_Pad1.15x1.40mm_HandSolder, symbol Device:C_Small
- removed J1: AN14, Connector_PinHeader_2.54mm:PinHeader_1x03_P2.54mm_Vertical, symbol Connector_Generic:Conn_01x03
- removed J10: SPI1_AUX, Connector_PinHeader_2.54mm:PinHeader_1x06_P2.54mm_Vertical, symbol Connector_Generic:Conn_01x06
- removed J11: I2C2_AUX, Connector_PinHeader_2.54mm:PinHeader_1x04_P2.54mm_Vertical, symbol Connector_Generic:Conn_01x04
- removed J2: GPIO1, Connector_PinHeader_2.54mm:PinHeader_1x03_P2.54mm_Vertical, symbol Connector_Generic:Conn_01x03
- removed J3: GPIO2, Connector_PinHeader_2.54mm:PinHeader_1x03_P2.54mm_Vertical, symbol Connector_Generic:Conn_01x03
- removed J4: GPIO3, Connector_PinHeader_2.54mm:PinHeader_1x03_P2.54mm_Vertical, symbol Connector_Generic:Conn_01x03
- removed J5: AN8, Connector_PinHeader_2.54mm:PinHeader_1x03_P2.54mm_Vertical, symbol Connector_Generic:Conn_01x03
- removed J6: AN9, Connector_PinHeader_2.54mm:PinHeader_1x03_P2.54mm_Vertical, symbol Connector_Generic:Conn_01x03
- removed J7: AN15, Connector_PinHeader_2.54mm:PinHeader_1x03_P2.54mm_Vertical, symbol Connector_Generic:Conn_01x03
- removed J8: Programming, Connector_PinHeader_2.54mm:PinHeader_1x06_P2.54mm_Vertical, symbol Connector_Generic:Conn_01x06
- removed J9: UART6_AUX, Connector_PinHeader_2.54mm:PinHeader_1x06_P2.54mm_Vertical, symbol Connector_Generic:Conn_01x06
- removed JP1, JP10, JP2, JP23, JP24, JP3, JP4, JP5, JP6: SolderJumper_3_Bridged12, Jumper:SolderJumper-3_P1.3mm_Bridged12_Pad1.0x1.5mm, symbol Jumper:SolderJumper_3_Bridged12
- removed JP11, JP14, JP15, JP16, JP17, JP18, JP19, JP20, JP21, JP22, JP7, JP8, JP9: SolderJumper_2_Bridged, Jumper:SolderJumper-2_P1.3mm_Bridged_Pad1.0x1.5mm, symbol Jumper:SolderJumper_2_Bridged
- removed JP12, JP13: SolderJumper_2_Open, Jumper:SolderJumper-2_P1.3mm_Open_Pad1.0x1.5mm, symbol Jumper:SolderJumper_2_Open
- removed R10, R15, R16, R17, R4, R5, R9: 1k, Resistor_SMD:R_0805_2012Metric_Pad1.15x1.40mm_HandSolder, symbol Device:R_Small
- removed R11, R14: 10k, Resistor_SMD:R_0805_2012Metric_Pad1.15x1.40mm_HandSolder, symbol Device:R_Small
- removed SW1: RESET_BP, Button_Switch_THT:SW_TH_Tactile_Omron_B3F-10xx, symbol Switch:SW_Push_Dual_x2
- removed SW2: WKP_BP, Button_Switch_THT:SW_TH_Tactile_Omron_B3F-10xx, symbol Switch:SW_Push_Dual_x2
- removed TP1: TestPoint, TestPoint:TestPoint_Pad_D1.5mm, symbol Connector:TestPoint
- removed U1: STM32F405RGTx, Package_QFP:LQFP-64_10x10mm_P0.5mm, symbol MCU_ST_STM32F4:STM32F405RGTx
- added C4, C9: 100nF, Capacitor_SMD:C_0805_2012Metric_Pad1.15x1.40mm_HandSolder, symbol Device:C_Small
- added SW1, SW2, SW3: DIP-BUTTON_2P-6.0X3.0X4.3MM_, Button_Switch_THT:SW_PUSH_6mm_H5mm, symbol OPL_Switch:DIP-BUTTON_2P-6.0X3.0X4.3MM_
- added U1: STM32F401RETx, Package_QFP:LQFP-64_10x10mm_P0.5mm, symbol MCU_ST_STM32F4:STM32F401RETx
- C1: value 100nF -> 18pF; LCSC C49678 -> C1797
- C6: value 2.2uF -> 4.7uF
- H1, H2, H3, H4: footprint MountingHole:MountingHole_2.7mm_M2.5 -> MountingHole:MountingHole_3.2mm_M3
- R2, R3: value 1k -> 10k; Catalog (none) -> Basic; LCSC (none) -> C17714
- R8: value Unpopulated -> 1k
- renumbered C11 to C10, C12 to C11, C13 to C12, C4 to C3, C9 to C8, R12 to R4, R13 to R5
Connections:
- net labels added: ADC_ML_SENSE, ADC_MR_SENSE, AUX_GPIO_1, AUX_GPIO_2, AUX_SPI_INT, AUX_UART_RX, AUX_UART_TX, BATT_ADC, BOOT0, BOOT1_BP2, BP1, DRV_EN, I2C_AUX_INT, I2C_AUX_SCL, I2C_AUX_SDA, NRF_SPI_MISO, NRF_SPI_MOSI, NRF_SPI_SCK, PWM_ML_H, PWM_ML_L, PWM_MR_H, PWM_MR_L, SPI_AUX_MISO, SPI_AUX_MOSI, SPI_AUX_NSS, SPI_AUX_SCK, SWCLK, SWIO, USB_DM, USB_DP, USB_VBUS, VL53l0_I2C_SCL, VL53l0_I2C_SDA
- net labels removed: +5V, ADC1_14, ADC1_15, ADC1_8, ADC1_9, FTDI_CTS, FTDI_RTS, FTDI_RX, FTDI_TX, I2C1_SCL, I2C1_SDA, I2C2_SCL, I2C2_SDA, ML_PWM_H, ML_PWM_L, MPU_FSYNC, MR_PWM_H, MR_PWM_L, SPI1_MISO, SPI1_MOSI, SPI1_NSS, SPI1_SCK, SPI2_MISO, SPI2_MOSI, SPI2_SCK, Servo1, Servo2, Servo3, TCK, TMS, UART6_RX, UART6_TX
- wire segments 301 -> 144
- no-connect marks 3 -> 0
Other:
- note added: "- 1x 100nF Cap for each VDD pin\n - 1x 10uF tantalum or ceramic for the chip\n - 1x 100nF for VBAT\n - 1x 100nF Ceramic + 1x 1uF tantalum or ceramic for VDDA/VREF"
- note added: "DONE:\n - Current sensing from driver chip needs to be connected to ADC pins\n - Battery monitoring (bridge divider to ADC pin)\n - PB2 is BOOT1 pin, look into it\n - change ALEDs pin to PC12 (SPI3 MOSI)\n - DRV8833 nSLEEP to NRST doesn't work, put it on a GPIO instead\n - Fix UART TX/RX Inversion on FTDI port\n - Fix UART TX/RX Inversion on AUX port\n - Add a jumper for motor power\n - Separate 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"
- note added: "TODO:\n - Remove optimization for JLCPCB PCBA service\n - Change default MCU for STM32F401\n - Change Button footprint\n - Add diode between power levels\n - Investigate why VBAT in back driven from 5V/3V3?\n - Less bright LEDs\n - Move TIM2 away from PA15 (default state high)\n - Change programaming connector interface (try to find a "standard online")\n - Move Mot/Coder header to the side of th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"
- note removed: "DONE:\n - Add a jumper for motor power\n - Separate Shield and Ground from USB connector"
- note removed: "STM32F4x1 compatibility:\n - Unpopulate C and close solder-jumper to VCAP_1 (pin 31) and VCAP_2 (pin 47)\n - Populate PB11 (pin 30) C"
- note removed: "SWCLK"
- note removed: "SWIO"
- note removed: "TODO:\n - Change Button footprint\n - Add diode between power levels\n - Investigate why VBAT in back driven from 5V/3V3?\n - Less bright LEDs\n - Move TIM2 away from PA15 (default state high)\n - Move Mot/Coder header to the side of th motors (with mirrored orientation)\n - Add 2 ALED in front and move button\n - Add 1/2 ALED in the back\n - Wider holes for battery\n - Better positions for stand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"
- moved on the sheet: D1, D2, R4, R5
