File: Electronics/PRoMo_v0_2/Power.sch (KiCad schematic (older format))
At the start: 22 parts, among them J18 Conn_01x02, J19 Conn_02x02_Counter_Clockwise, J20 Conn_02x02_Counter_Clockwise, J21 AUX_IN, J22 AUX_OUT, SW3 SW_SPDT, U8 LM2596S-5, U9 AMS1117-3.3

Commit message: Start working on HW v0.2
Parts:
- renumbered C33 to C25, C34 to C26, C35 to C27, D16 to D10, D17 to D11, D18 to D12, D14 to D8, D15 to D9, J20 to J10, J21 to J11, J22 to J12, J18 to J8, J19 to J9, R21 to R11, R22 to R12, R23 to R13, R24 to R14, SW3 to SW4
