File: Electronics/PRoMo_v0_2/Sensors.sch (KiCad schematic (older format))
At the start: 28 parts, among them J12 Conn_01x02, J13 Conn_01x02, J14 Conn_01x02, J15 Conn_01x02, U2 VL53l0x_breakout, U3 VL53l0x_breakout, U4 VL53l0x_breakout, U5 VL53l0x_breakout, U6 MPU-6050

Commit message: Start working on HW v0.2
Parts:
- added J5: Conn_01x03, Connector_PinHeader_2.54mm:PinHeader_1x03_P2.54mm_Vertical, symbol Connector_Generic:Conn_01x03
- renumbered C15 to C13, C16 to C14, C18 to C15, C20 to C16, C22 to C17, C26 to C18, C27 to C19, C28 to C20, C29 to C21, D6 to D5, D8 to D6, D10 to D7, J12 to J1, J13 to J2, J14 to J3, J15 to J4, JP25 to JP1, TP2 to TP1, TP3 to TP2, TP7 to TP3
Connections:
- net +5V: now also J5.1 (Pin_1)
- net GND: now also J5.3 (Pin_3)
- net at D7.4 (DOUT), TP3.1: now also J5.2 (Pin_2)
- net I2C1_SCL renamed VL53l0_I2C_SCL
- net I2C1_SDA renamed VL53l0_I2C_SDA
- net I2C2_SCL renamed AUX_I2C_SCL
- net I2C2_SDA renamed AUX_I2C_SDA
Other:
- note added: "Replace jumper with open solder bridge?"
- moved on the sheet: JP1, TP1, TP2, TP3, TP4
